File: PCB/SCC-Switch.kicad_sch (KiCad schematic)
At the start: 11 parts, among them J1 USB_C_Receptacle_USB2.0_14P, U1 KSZ8895RQXI, U2 AP63203WU

Commit message: More Power Ciruits, Add MCU, Add Switch Chip
Parts:
- removed U1: KSZ8895RQXI, PQFP-128_MQL_MCH, symbol Interface_Ethernet:KSZ8895RQXI
- added C6: 10 µF, symbol Device:C
- added C7: 0.1 µF, symbol Device:C
- added J2, J3, J4, J5, J6: RJ45, symbol Connector:RJ45
- added U1: KSZ9897STXC, TQFP-EP128_TX_MCH, symbol Interface_Ethernet:KSZ9897STXC
- added U3: Raspberry_Pi_Pico, ScottoKeebs_MCU:Raspberry_Pi_Pico, symbol ScottoKeebs:MCU_Raspberry_Pi_Pico
Connections:
- net +5V: now also C6.1, C7.1, U3.39 (VSYS)
- net GND: now also C6.2, C7.2, U1.46 (GND), U1.47 (GND)
- new net +1V0: U1.11 (DVDDL), U1.14 (AVDDL), U1.19 (AVDDL), U1.20 (TXRX2P_D), U1.23 (DVDDL), U1.3 (AVDDL), U1.30 (AVDDL), U1.36 (AVDDL), U1.41 (AVDDL), U1.45 (DVDDL), U1.56 (DVDDL)
- new net +3V3: U1.10 (AVDDH), U1.22 (AVDDH), U1.33 (AVDDH), U1.44 (AVDDH), U1.61 (VDDIO)
Other:
- note added: "MCU"
- note added: "Power"
